File: led-heart.sch (EAGLE design)
At the start: 65 parts, among them IC1 FT232RL, IC2 MSP430F149, Q1 8mhz, T1 MMBT3904, T2 MMBT3904, X1 USB_MINI-B

Commit message: release, fix schematic, pcb, silk, docs
Parts:
- removed D1: LIS302DL, colibri:LIS302DL
- removed R5: 100k, colibri:RES
- removed T1, T2: MMBT3904, transistor:MMBT3904LT1-NPN-SOT23-BEC
- added IC3: LIS302DL, netcat:LIS302DL
- added LOGO1: LOGO2, netcat:LOGO2
- added Q2: MMBT3904, netcat:NPNSOT23
- added QZ1: 8MHz, netcat:QUARTZHC49
- added R2: 4.7k, netcat:RESR0805
- added R3: 100k, netcat:RESR0805
- B1: device Di:BATTERY -> netcat:CR2032
- C1, C2: value 0,1u -> 100n; device colibri:CAP -> netcat:CAP0805
- C3: value 10n -> 12p; device colibri:CAP -> netcat:CAP0805
- C4: device colibri:CAP -> netcat:CAP0805
- C5: value 12p -> 100n; device colibri:CAP -> netcat:CAP0805
- IC1: device ftdichip:FT232RL -> netcat:FT232RL
- IC2: value MSP430F149 -> MSP430F249; device texas:MSP430F149 -> netcat:MSP430F249
- LED10, LED11, LED12, LED13, LED14, LED15, LED16, LED17, LED18, LED19, LED20, LED21, LED22, LED23, LED24, LED25, LED26, LED27, LED28, LED29, LED3, LED30, LED31, LED32, LED33, LED34, LED35, LED36, LED37, LED38, LED39, LED4, LED40, LED41, LED42, LED43, LED44, LED45, LED46, LED47, LED48, LED49, LED5, LED50, LED6, LED7, LED8, LED9: device led:LEDCHIP-LED0603 -> netcat:LED0603
- Q1: value 8mhz -> MMBT3904; device crystal:CRYSTALSM49 -> netcat:NPNSOT23
- R1: value 0 -> 4.7k; device colibri:RES -> netcat:RESR0805
- R4: device colibri:RES -> netcat:RESR0805
- U$1: device Di:TOUCH_SENSOR -> netcat:TOUCH_SENSOR
- X1: value USB_MINI-B -> USB-MINI-B; device colibri:USB_MINI-B -> netcat:USB-MINI-B
Connections:
- removed net VCCINT: B1.PLUS, D1.CS, D1.SDO, D1.VCC@1, D1.VDDIO, IC2.AVCC, IC2.DVCC, R1.1, R4.1
- new net VCC: B1.PLUS, C5.1, IC2.AVCC, IC2.DVCC, IC3.CS, IC3.SDO, IC3.VCC@0, IC3.VDDIO, R1.1, R2.1, R4.1
- net !BSL_RTS: no longer C3.1
- net EN1: now also Q2.B; no longer T2.B
- net EN2: now also Q1.B; no longer T1.B
- net GND: now also C3.1, C5.2, IC3.GND@0, Q1.E, Q2.E, R3.1; no longer C3.2, C5.1, D1.GND@0, D1.GND@1, D1.GND@2, D1.GND@3, D1.GND@4, R5.1, T1.E, T2.E
- net I2C_SCL: now also IC3.SCL, R2.2; no longer D1.SCL, IC2.P3.2
- net I2C_SDA: now also IC3.SDA/SDI, R1.2; no longer D1.SDA/SDI
- net N$10: now also Q2.C; no longer T2.C
- net N$11: now also C4.2, QZ1.1; no longer C5.2, Q1.1
- net N$12: now also R3.2; no longer R5.2
- net N$6: no longer R1.2
- net N$8: now also C3.2, QZ1.2; no longer C4.2, Q1.2
- net N$9: now also Q1.C; no longer T1.C
Other:
- moved on the sheet: B1, IC1, IC2, LED10, LED11, LED12, LED13, LED14, LED15, LED16, LED17, LED18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

Commit message: new design, qfn packages, buzzer for sound
Parts:
- removed IC3: LIS302DL, netcat:LIS302DL
- removed R1, R2: 4.7k, netcat:RESR0805
- removed R3, R4: 100k, netcat:RESR0805
- added BZ1: (no value), netcat:BUZZERHYG2575
- added L1: 10uH, netcat:L-1812
- added Q3: IRLML2402, netcat:MOSFET_NSOT23
- added R5: 100k, netcat:RESR0402
- added VD1: 4148, netcat:DIODE-SOD123
- C1: value 100n -> 0.1u; device netcat:CAP0805 -> netcat:CAP0402
- C2: value 100n -> 10u; device netcat:CAP0805 -> netcat:CAP0603
- C3: value 12p -> 10u; device netcat:CAP0805 -> netcat:CPOL-EUSMCA
- C4: device netcat:CAP0805 -> netcat:CAP0402
- C5: value 100n -> 12p; device netcat:CAP0805 -> netcat:CAP0402
- IC1: value FT232RL -> FT232RQ; device netcat:FT232RL -> netcat:FT232RQ
- IC2: value MSP430F249 -> MSP430F2370; device netcat:MSP430F249 -> netcat:MSP430F2370
- Q1, Q2: value MMBT3904 -> IRLML2402; device netcat:NPNSOT23 -> netcat:MOSFET_NSOT23
- QZ1: value 8MHz -> 8mhz; device netcat:QUARTZHC49 -> netcat:QUARTZ_GND3225
- X1: value USB-MINI-B -> USBMICRO_B; device netcat:USB-MINI-B -> netcat:USBMICRO_B
Connections:
- net N$34 renamed 5V
- net N$6 renamed VCCIO
- removed net BSL_RXD: IC1.RXD, IC2.P1.1
- removed net BSL_TXD: IC1.TXD, IC2.P2.2
- removed net I2C_SCL: IC2.P3.3, IC3.SCL, R2.2
- removed net I2C_SDA: IC2.P3.1, IC3.SDA/SDI, R1.2
- removed net N$1: IC1.USBDP, X1.DP
- removed net N$10: LED27.C, LED28.C, LED29.C, LED30.C, LED31.C, LED32.C, LED33.C, LED34.C, LED35.C, LED36.C, LED37.C, LED38.C, LED39.C, LED40.C, LED41.C, LED42.C, LED43.C, LED44.C, LED45.C, LED46.C, LED47.C, LED48.C, LED49.C, LED50.C, Q2.C
- removed net N$11: C4.2, IC2.XOUT/TCLK, QZ1.1
- removed net N$12: IC2.P1.0, R3.2, U$1.CON
- removed net N$33: IC1.USBDM, X1.DM
- removed net N$8: C3.2, IC2.XIN, QZ1.2
- removed net N$9: LED10.C, LED11.C, LED12.C, LED13.C, LED14.C, LED15.C, LED16.C, LED17.C, LED18.C, LED19.C, LED20.C, LED21.C, LED22.C, LED23.C, LED24.C, LED25.C, LED26.C, LED3.C, LED4.C, LED5.C, LED6.C, LED7.C, LED8.C, LED9.C, Q1.C
- removed net VCC: B1.PLUS, C5.1, IC2.AVCC, IC2.DVCC, IC3.CS, IC3.SDO, IC3.VCC@0, IC3.VDDIO, R1.1, R2.1, R4.1
- new net 3.3V: B1.PLUS, C3.+, IC2.AVCC, IC2.DVCC, L1.P$1
- new net BOOST: L1.P$2, VD1.A
- new net LINE1: LED27.C, LED28.C, LED29.C, LED30.C, LED31.C, LED32.C, LED33.C, LED34.C, LED35.C, LED36.C, LED37.C, LED38.C, LED39.C, LED40.C, LED41.C, LED42.C, LED43.C, LED44.C, LED45.C, LED46.C, LED47.C, LED48.C, LED49.C, LED50.C, Q1.D
- new net LINE2: LED10.C, LED11.C, LED12.C, LED13.C, LED14.C, LED15.C, LED16.C, LED17.C, LED18.C, LED19.C, LED20.C, LED21.C, LED22.C, LED23.C, LED24.C, LED25.C, LED26.C, LED3.C, LED4.C, LED5.C, LED6.C, LED7.C, LED8.C, LED9.C, Q3.D
- new net SENS: IC2.P1.4/SMCLK/TCK, R5.2, U$1.CON
- new net SENS2: IC2.P1.5/TA0/TMS, R5.1
- new net SND: IC2.P1.2/TA1, Q2.G
- new net USB+DP: IC1.USBDP, X1.D+
- new net USB_DM: IC1.USBDM, X1.D-
- new net V_SND: BZ1.P, Q2.D, VD1.C
- new net XIN: C5.2, IC2.XIN/P2.6, QZ1.1
- new net XOUT: C4.2, IC2.XOUT/P2.7, QZ1.2
- net !BSL_RTS: now also IC2.!RST!/NMI; no longer IC2.!RTS!/NMI, R4.2
- net EN1: now also IC1.RXD, IC2.P1.1/TA0, Q1.G; no longer IC2.P1.2, Q2.B
- net EN2: now also IC2.P1.3/TA2, Q3.G; no longer IC2.P1.3, Q1.B
- net GND: now also BZ1.M, C3.-, C5.1, IC2.D/AVSS, Q1.S, Q2.S, Q3.S, QZ1.GND; no longer C3.1, C5.2, IC2.AVSS, IC2.DVSS, IC3.GND@0, Q1.E, Q2.E, R3.1
- net LED0: now also IC2.P2.0/ACLK/A0/OA0I0; no longer IC2.P4.0
- net LED1: now also IC2.P2.1/TAINCLK/SMCLK/A1/OA0O; no longer IC2.P4.1
- net LED10: now also IC2.P3.2/UCB0SOMI/UCB0SCL; no longer IC2.P5.2
- net LED11: now also IC2.P3.3/UCB0CLK/UCA0STE; no longer IC2.P5.3
- net LED12: now also IC2.P3.4/UCA0TXD/UCA0SIMO; no longer IC2.P5.4
- net LED13: now also IC2.P3.5/UCA0RXD/UCA0SOMI; no longer IC2.P5.5
- net LED14: now also IC2.P3.6/A6/OA0I2; no longer IC2.P5.6
- net LED15: now also IC2.P3.7/A7/OA1I2; no longer IC2.P5.7
- net LED16: now also IC2.P4.0/TB0; no longer IC2.P6.0
- net LED17: now also IC2.P4.1/TB1; no longer IC2.P6.1
- net LED18: now also IC2.P4.2/TB2; no longer IC2.P6.2
- net LED19: now also IC2.P4.3/TB0/A12/OA0O; no longer IC2.P6.3
- net LED2: now also IC1.TXD, IC2.P2.2/TA0/A2/OA0I1; no longer IC2.P4.2
- net LED20: now also IC2.P4.4/TB1A13/OA1O; no longer IC2.P6.4
- net LED21: now also IC2.P4.5/TB2A14/OA0I3; no longer IC2.P6.5
- net LED22: now also IC2.P4.6/TBOUTHA15/OA1I3; no longer IC2.P6.6
- net LED23: now also IC2.P4.7/TBCLK; no longer IC2.P6.7
- net LED3: now also IC2.P2.3/TA1/A3/VREF-/VEREF-/OA1I1/OA1O; no longer IC2.P4.3
- net LED4: now also IC2.P2.4/TA2/A4/VREF+/VEREF+/OA1I0; no longer IC2.P4.4
- net LED5: now also IC2.P2.5/ROSC; no longer IC2.P4.5
- net LED6: now also IC2.P1.6/TA1/TDI/TCLK; no longer IC2.P4.6
- net LED7: now also IC2.P1.7/TA2/TDO/TDI; no longer IC2.P4.7
- net LED8: now also IC2.P3.0/UCB0STE/UCA0CLK/A5; no longer IC2.P5.0
- net LED9: now also IC2.P3.1/UCB0SIMO/UCB0SDA; no longer IC2.P5.1
Other:
- moved on the sheet: B1, C1, C2, C4, C5, IC1, LED10, LED11, LED12, LED13, LED14, LED15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
